File: VGA.kicad_pcb (KiCad board)
At the start: 2 copper layers, 41.9 x 27.9 mm, 20 parts, among them J1 Conn_01x16, J2 DB15_Female_HighDensity

Commit message: Small changes
Other:
- board text added: "@hasecilu"
- board text added: "v 1.2"
- board text removed: "Ulices AH"
- board text removed: "v 1.1"
